Commit message: robot 1 completed yay

File: milestone5_ws/src/robots_viz/urdf/robot1.urdf.xacro (robot description, xacro)
@@ -7,8 +7,8 @@
   <xacro:property name="L2_size" value="0.05" />
   <xacro:property name="L3" value="0.08" />
-  <xacro:property name="L3_size" value="0.05" />
-  <xacro:property name="L4" value="0.06" />
-  <xacro:property name="L4_size" value="0.03" />
-  <xacro:property name="ee_size" value="0.04" />
+  <xacro:property name="L3_size" value="0.03" />
+  <xacro:property name="L4" value="0.05" />
+  <xacro:property name="L4_size" value="0.02" />
+  <xacro:property name="ee_size" value="0.03" />
   <xacro:property name="J1MIN" value="-0.10" />
   <xacro:property name="J1MAX" value="0.10" />
@@ -24,10 +24,9 @@
   </material>
   <link name="world" />
-  <link name="base" />
   <link name="link1">
     <visual name="link1">
-      <origin xyz="0 0 ${L1/2}" />
+      <origin xyz="0 0 ${(L1+J1MAX+(L2_size/2))/2}" />
       <geometry>
-        <box size="${L1_size} ${L1_size} ${L1}" />
+        <box size="${L1_size} ${L1_size} ${L1+J1MAX+(L2_size/2)}" />
       </geometry>
       <material name="blue" />
@@ -36,7 +35,7 @@
   <link name="link2">
     <visual name="link2">
-      <origin rpy="0 ${pi/2} 0" xyz="${L2/2} 0 0" />
+      <origin rpy="${-pi/2} 0 0" xyz="0 ${(L2+J2MAX+(L3_size/2))/2} 0" />
       <geometry>
-        <box size="${L2_size} ${L2_size} ${L2}" />
+        <box size="${L2_size} ${L2_size} ${L2+J2MAX+(L3_size/2)}" />
       </geometry>
       <material name="blue" />
@@ -45,5 +44,5 @@
   <link name="link3">
     <visual name="link3">
-      <origin rpy="${pi/2} 0 0" xyz="0 0 0 " />
+      <origin rpy="${pi/2} 0 0" xyz="0 ${-(-L3/2)} 0 " />
       <geometry>
         <box size="${L3_size} ${L3_size} ${L3}" />
@@ -54,7 +53,7 @@
   <link name="link4">
     <visual name="link4">
-      <origin rpy="${pi/2} 0 0" xyz="0 0 0 " />
+      <origin rpy="0 0 0" xyz="0 0 ${(L4-J3MAX)/2} " />
       <geometry>
-        <box size="${L4_size} ${L4_size} ${L4}" />
+        <box size="${L4_size} ${L4_size} ${L4+J3MAX}" />
       </geometry>
       <material name="blue" />
@@ -70,13 +69,8 @@
     </visual>
   </link>
-  <joint name="base_in_world" type="fixed">
+  <joint name="link1_in_world" type="fixed">
     <parent link="world" />
-    <child link="base" />
-    <origin xyz="${-L2} ${(ee_size/2)+(L4)+L3} 0" />
-  </joint>
-  <joint name="link1_in_base" type="fixed">
-    <parent link="base" />
     <child link="link1" />
-    <origin xyz="0 0 0" />
+    <origin rpy="0 0 ${-pi/2}" xyz="${-L2} ${(ee_size/2)+(L4)+L3} 0" />
   </joint>
   <joint name="joint1" type="prismatic">
@@ -90,6 +84,6 @@
     <parent link="link2" />
     <child link="link3" />
-    <origin rpy="0 0 0" xyz="${L2} 0 0" />
-    <axis xyz="1 0 0" />
+    <origin rpy="${-pi/2} ${-pi/2} 0" xyz="0 ${L2} 0" />
+    <axis xyz="0 0 1" />
     <limit lower="${J2MIN}" upper="${J2MAX}" effort="1" velocity="1" />
   </joint>
@@ -97,6 +91,6 @@
     <parent link="link3" />
     <child link="link4" />
-    <origin rpy="0 0 0" xyz="0 ${-L3} 0" />
-    <axis xyz="0 1 0" />
+    <origin rpy="${-pi/2} 0 0" xyz="0 ${L3} 0" />
+    <axis xyz="0 0 1 " />
     <limit lower="${J3MIN}" upper="${J3MAX}" effort="1" velocity="1" />
   </joint>
@@ -104,5 +98,5 @@
     <parent link="link4" />
     <child link="ee" />
-    <origin xyz="0 ${-L4} 0" rpy="0 0 0" />
+    <origin xyz="0 0 ${L4+ee_size/2}" rpy="0 0 0" />
   </joint>
 </robot>

File: milestone5_ws/src/robots_viz/urdf/robot3.urdf.xacro (robot description, xacro)
@@ -27,7 +27,7 @@
   <link name="link1">
     <visual name="link1">
-      <origin xyz="0 0 ${L1/2}" />
+      <origin xyz="0 0 ${(L1+J1MAX+(L2_size/2))/2}" />
       <geometry>
-        <box size="${L1_size} ${L1_size} ${L1}" />
+        <box size="${L1_size} ${L1_size} ${L1+J1MAX+L2_size/2}" />
       </geometry>
       <material name="blue" />
@@ -54,5 +54,5 @@
   <link name="link4">
     <visual name="link4">
-      <origin rpy="0 ${pi/2} 0" xyz="${L4/2} 0 0 " />
+      <origin rpy="0 0 0" xyz="0 0 ${L4/2} " />
       <geometry>
         <box size="${L4_size} ${L4_size} ${L4}" />
@@ -97,6 +97,6 @@
     <parent link="link3" />
     <child link="link4" />
-    <origin rpy="0 0 0" xyz="${L3} 0 0" />
-    <axis xyz="1 0 0" />
+    <origin rpy="0 ${pi/2} 0" xyz="${L3} 0 0" />
+    <axis xyz="0 0 1" />
     <limit lower="${J3MIN}" upper="${J3MAX}" effort="1" velocity="1" />
   </joint>
@@ -104,5 +104,5 @@
     <parent link="link4" />
     <child link="ee" />
-    <origin xyz="${L4} 0 0" rpy="0 0 0" />
+    <origin xyz="0 0 ${L4}" rpy="0 ${-pi/2} 0" />
   </joint>
 </robot>
