Commit message: robot 1 and 3 basics complete

File: milestone5_ws/src/robots_viz/urdf/robot3.urdf.xacro (robot description, xacro)
@@ -1,20 +1,20 @@
 <?xml version="1.0" encoding="UTF-8"?>
 <!DOCTYPE xml>
-<robot xmlns:xacro="http://www.ros.org/wiki/xacro" name="robot1">
-  <xacro:property name="L1" value="0.25" />
+<robot xmlns:xacro="http://www.ros.org/wiki/xacro" name="robot3">
+  <xacro:property name="L1" value="0.20" />
   <xacro:property name="L1_size" value="0.05" />
-  <xacro:property name="L2" value="0.20" />
+  <xacro:property name="L2" value="0.08" />
   <xacro:property name="L2_size" value="0.05" />
-  <xacro:property name="L3" value="0.08" />
+  <xacro:property name="L3" value="0.06" />
   <xacro:property name="L3_size" value="0.05" />
   <xacro:property name="L4" value="0.06" />
   <xacro:property name="L4_size" value="0.03" />
   <xacro:property name="ee_size" value="0.04" />
-  <xacro:property name="J1MIN" value="-0.10" />
-  <xacro:property name="J1MAX" value="0.10" />
-  <xacro:property name="J2MIN" value="-0.07" />
-  <xacro:property name="J2MAX" value="0.07" />
-  <xacro:property name="J3MIN" value="-0.05" />
-  <xacro:property name="J3MAX" value="0.05" />
+  <xacro:property name="J1MIN" value="-0.08" />
+  <xacro:property name="J1MAX" value="0.08" />
+  <xacro:property name="J2MIN" value="${-pi/2}" />
+  <xacro:property name="J2MAX" value="${pi/2}" />
+  <xacro:property name="J3MIN" value="-0.04" />
+  <xacro:property name="J3MAX" value="0.04" />
   <material name="blue">
     <color rgba="0.2 0.4 0.65 1" />
@@ -45,5 +45,5 @@
   <link name="link3">
     <visual name="link3">
-      <origin rpy="${pi/2} 0 0" xyz="0 0 0 " />
+      <origin rpy="0 ${pi/2} 0" xyz="${L3/2} 0 0 " />
       <geometry>
         <box size="${L3_size} ${L3_size} ${L3}" />
@@ -54,5 +54,5 @@
   <link name="link4">
     <visual name="link4">
-      <origin rpy="${pi/2} 0 0" xyz="0 0 0 " />
+      <origin rpy="0 ${pi/2} 0" xyz="${L4/2} 0 0 " />
       <geometry>
         <box size="${L4_size} ${L4_size} ${L4}" />
@@ -73,5 +73,5 @@
     <parent link="world" />
     <child link="base" />
-    <origin xyz="${-L2} ${(ee_size/2)+(L4)+L3} 0" />
+    <origin xyz="${-(L4+L3+L2)} 0 0" />
   </joint>
   <joint name="link1_in_base" type="fixed">
@@ -87,9 +87,9 @@
     <limit lower="${J1MIN}" upper="${J1MAX}" effort="1" velocity="1" />
   </joint>
-  <joint name="joint2" type="prismatic">
+  <joint name="joint2" type="revolute">
     <parent link="link2" />
     <child link="link3" />
     <origin rpy="0 0 0" xyz="${L2} 0 0" />
-    <axis xyz="1 0 0" />
+    <axis xyz="0 0 1" />
     <limit lower="${J2MIN}" upper="${J2MAX}" effort="1" velocity="1" />
   </joint>
@@ -97,6 +97,6 @@
     <parent link="link3" />
     <child link="link4" />
-    <origin rpy="0 0 0" xyz="0 ${-L3} 0" />
-    <axis xyz="0 1 0" />
+    <origin rpy="0 0 0" xyz="${L3} 0 0" />
+    <axis xyz="1 0 0" />
     <limit lower="${J3MIN}" upper="${J3MAX}" effort="1" velocity="1" />
   </joint>
@@ -104,5 +104,5 @@
     <parent link="link4" />
     <child link="ee" />
-    <origin xyz="0 ${-L4} 0" rpy="0 0 0" />
+    <origin xyz="${L4} 0 0" rpy="0 0 0" />
   </joint>
 </robot>

Commit message: robot 3 also finished

File: milestone5_ws/src/robots_viz/urdf/robot3.urdf.xacro (robot description, xacro)
@@ -45,5 +45,5 @@
   <link name="link3">
     <visual name="link3">
-      <origin rpy="0 ${pi/2} 0" xyz="${L3/2} 0 0 " />
+      <origin rpy="${pi/2} 0 0" xyz="0 ${L3/2} 0 " />
       <geometry>
         <box size="${L3_size} ${L3_size} ${L3}" />
@@ -54,7 +54,7 @@
   <link name="link4">
     <visual name="link4">
-      <origin rpy="0 0 0" xyz="0 0 ${L4/2} " />
+      <origin rpy="0 0 0" xyz="0 0 ${(L4-J3MAX)/2} " />
       <geometry>
-        <box size="${L4_size} ${L4_size} ${L4}" />
+        <box size="${L4_size} ${L4_size} ${L4+J3MAX}" />
       </geometry>
       <material name="blue" />
@@ -90,5 +90,5 @@
     <parent link="link2" />
     <child link="link3" />
-    <origin rpy="0 0 0" xyz="${L2} 0 0" />
+    <origin rpy="0 0 ${-pi/2}" xyz="${L2} 0 0" />
     <axis xyz="0 0 1" />
     <limit lower="${J2MIN}" upper="${J2MAX}" effort="1" velocity="1" />
@@ -97,5 +97,5 @@
     <parent link="link3" />
     <child link="link4" />
-    <origin rpy="0 ${pi/2} 0" xyz="${L3} 0 0" />
+    <origin rpy="${-pi/2} 0 0" xyz="0 ${L3} 0" />
     <axis xyz="0 0 1" />
     <limit lower="${J3MIN}" upper="${J3MAX}" effort="1" velocity="1" />
@@ -104,5 +104,5 @@
     <parent link="link4" />
     <child link="ee" />
-    <origin xyz="0 0 ${L4}" rpy="0 ${-pi/2} 0" />
+    <origin xyz="0 0 ${L4}" rpy="0 0 0" />
   </joint>
 </robot>
