Commit message: wx250s and 5.3 completed

File: milestone5_ws/src/wx250s_viz/urdf/wx250s.urdf.xacro (robot description, xacro)
@@ -8,4 +8,6 @@
   <xacro:property name="L2" value="0.25" />
   <xacro:property name="L2radius" value="0.05" />
+  <xacro:property name="Lfixed" value="0.10" />
+  <xacro:property name="Lfixedradius" value="0.05" />
   <xacro:property name="L3" value="0.17155" />
   <xacro:property name="L3radius" value="0.05" />
@@ -59,4 +61,13 @@
       <geometry>
         <cylinder radius="${L2radius}" length="${L2}" />
+      </geometry>
+      <material name="blue" />
+    </visual>
+  </link>
+  <link name="linkfixed">
+    <visual name="linkfixed">
+      <origin rpy="${pi/2} 0 0" xyz="0 0 0" />
+      <geometry>
+        <cylinder radius="${Lfixedradius}" length="${Lfixed}" />
       </geometry>
       <material name="blue" />
@@ -127,8 +138,13 @@
     <limit lower="${J2MIN}" upper="${J2MAX}" effort="1" velocity="1" />
   </joint>
+  <joint name="jointfixed" type="fixed">
+    <parent link="link2" />
+    <child link="linkfixed" />
+    <origin rpy="0 0 0" xyz="0 0 ${L2}" />
+  </joint>
   <joint name="joint3" type="revolute">
-    <parent link="link2" />
+    <parent link="linkfixed" />
     <child link="link3" />
-    <origin rpy="0 0 0" xyz="0.05 0 ${L2}" />
+    <origin rpy="0 0 0" xyz="0.05 0 0" />
     <axis xyz="0 1 0" />
     <limit lower="${J3MIN}" upper="${J3MAX}" effort="1" velocity="1" />

Commit message: milestone 5 complete

File: milestone5_ws/src/wx250s_viz/urdf/wx250s.urdf.xacro (robot description, xacro)
@@ -7,15 +7,15 @@
   <xacro:property name="L1radius" value="0.10" />
   <xacro:property name="L2" value="0.25" />
-  <xacro:property name="L2radius" value="0.05" />
+  <xacro:property name="L2radius" value="0.03" />
   <xacro:property name="Lfixed" value="0.10" />
   <xacro:property name="Lfixedradius" value="0.05" />
   <xacro:property name="L3" value="0.17155" />
-  <xacro:property name="L3radius" value="0.05" />
+  <xacro:property name="L3radius" value="0.03" />
   <xacro:property name="L4" value="0.07845" />
-  <xacro:property name="L4radius" value="0.055" />
+  <xacro:property name="L4radius" value="0.04" />
   <xacro:property name="L5" value="0.065" />
-  <xacro:property name="L5radius" value="0.05" />
+  <xacro:property name="L5radius" value="0.03" />
   <xacro:property name="L6" value="0.10915" />
-  <xacro:property name="L6radius" value="0.055" />
+  <xacro:property name="L6radius" value="0.04" />
   <xacro:property name="eesize" value="0.05" />
   <xacro:property name="J1MIN" value="${-pi}" />
@@ -135,5 +135,5 @@
     <child link="link2" />
     <origin rpy="0 0 0" xyz="0 0 ${L1}" />
-    <axis xyz="0 1 0" />
+    <axis xyz="0 -1 0" />
     <limit lower="${J2MIN}" upper="${J2MAX}" effort="1" velocity="1" />
   </joint>
@@ -147,5 +147,5 @@
     <child link="link3" />
     <origin rpy="0 0 0" xyz="0.05 0 0" />
-    <axis xyz="0 1 0" />
+    <axis xyz="0 -1 0" />
     <limit lower="${J3MIN}" upper="${J3MAX}" effort="1" velocity="1" />
   </joint>
@@ -161,5 +161,5 @@
     <child link="link5" />
     <origin rpy="0 0 0" xyz="${L4} 0 0" />
-    <axis xyz="0 1 0" />
+    <axis xyz="0 -1 0" />
     <limit lower="${J5MIN}" upper="${J5MAX}" effort="1" velocity="1" />
   </joint>
